Commit message: nav2 maybe

File: src/my_bot/description/lidar.xacro (robot description, xacro)
@@ -4,5 +4,5 @@
         <parent link="chassis"/>
         <child link="laser"/>
-        <origin xyz="0.05 0.05 0.07" rpy="0 0 0"/>
+        <origin xyz="0.05 -0.05 0.07" rpy="0 0 0"/>
     </joint>
     <link name="laser">
